File: D12.kicad_pcb (KiCad board)
At the start: 4 copper layers, 50.9 x 15.5 mm, 72 parts, among them IC1 DRV8847RTER, IC2 NCP730BM, J1 Conn_01x01, J2 Conn_01x01, J3 Conn_01x01, J4 Conn_01x01, J5 UDPI, J6 Conn_01x01, J7 Conn_01x01, J8 Conn_01x01, J9 Conn_01x01, Q1 BC857BDW1, Q2 BC847BDW1, U1 AVR-64DA32, U3 BNO055, U4 TPS22810DRVR

Commit message: Initial commit
Parts:
- removed IC1: DRV8847RTER, _Samac:QFN50P300X300X80-17N-D
- removed IC2: NCP730BM, Package_SON:WSON-6-1EP_2x2mm_P0.65mm_EP1x1.6mm_ThermalVias
- removed U4: TPS22810DRVR, Package_DFN_QFN:DFN-6-1EP_2x2mm_P0.65mm_EP1x1.6mm
- renumbered D5 to D3, D3 to D5, J8 to J1, J1 to J5, J5 to J7, J9 to J8, J7 to J9, R24 to R14, R7 to R21, R5 to R22, R25 to R23, R6 to R24, R4 to R25, R21 to R4, R14 to R5, R8 to R6, R22 to R7, R23 to R8, U3 to U2
Connections:
- C16 pad 1: Net-(C16-Pad1) -> (no net)
- R16 pad 1: Net-(IC1-Pad16) -> (no net)
- U1 pad 1: TRQ -> (no net)
- U1 pad 2: PWM2 -> (no net)
- U1 pad 3: PWM1 -> (no net)
- U1 pad 4: ~FAULT -> (no net)
Routing:
- net (no net): track 0.00 -> 56.3 mm
- net ~FAULT: track 14.5 -> 0.00 mm
- net PWM1: track 13.2 -> 0.00 mm
- net PWM2: track 11.9 -> 0.00 mm
- net TRQ: track 10.4 -> 0.00 mm
- net Net-(C16-Pad1): track 3.29 -> 0.00 mm
- net Net-(IC1-Pad16): track 3.06 -> 0.00 mm
- removed copper zone on B.Cu, net Net-(J5-Pad1)

Commit message: Initial commit
Parts:
- added IC1: DRV8847RTER, RTB:QFN50P300X300X80-17N-D, F.Cu at (68.0, -43.2)
- added IC2: NCP730BM, Package_SON:WSON-6-1EP_2x2mm_P0.65mm_EP1x1.6mm_ThermalVias, F.Cu at (82.1, -43.3)
- added U4: TPS22810DRVR, Package_DFN_QFN:DFN-6-1EP_2x2mm_P0.65mm_EP1x1.6mm, F.Cu at (79.0, -43.3)
- C16: value 47nF -> 100nF
- C20: value n.f. -> 100n/50V
- C7: value N x 100u/16V -> N x 47u/25V
- R4, R8: value 10k -> n.f.
Connections:
- C16 pad 1: (no net) -> Net-(C16-Pad1)
- R16 pad 1: (no net) -> Net-(IC1-Pad16)
- U1 pad 1: (no net) -> TRQ
- U1 pad 2: (no net) -> PWM2
- U1 pad 3: (no net) -> PWM1
- U1 pad 4: (no net) -> ~FAULT
Routing:
- net (no net): track 56.3 -> 0.00 mm
- net ~FAULT: track 0.00 -> 14.5 mm
- net PWM1: track 0.00 -> 13.2 mm
- net PWM2: track 0.00 -> 11.9 mm
- net TRQ: track 0.00 -> 10.4 mm
- net Net-(C16-Pad1): track 0.00 -> 3.29 mm
- net Net-(IC1-Pad16): track 0.00 -> 3.06 mm
